File: short-circuit-limiter/schematic/short-circuit-limiter.sch (KiCad schematic (older format))
At the start: 6 parts

Commit message: connect everything
Parts:
- removed P?: M1363, symbol M1363
- removed SW? (x2): SWITCH_DPST, symbol SWITCH_DPST
- removed U?: D2450, SSR, symbol D2450
- added C1: 10uF, Capacitors_ThroughHole:CP_Radial_D5.0mm_P2.50mm, symbol CP
- added MCU1: Industruino-1286, Pin_Headers:Pin_Header_Angled_1x23_Pitch1.27mm, symbol Industruino-1286
- added P1: M1363, Buttons_Switches_SMD:SW_DIP_x1_W5.9mm_Slide_Copal_CVS, symbol M1363
- added R1: 4.7K, Resistors_ThroughHole:R_Axial_DIN0207_L6.3mm_D2.5mm_P10.16mm_Horizontal, symbol R
- added R2, R3: 470K, Resistors_ThroughHole:R_Axial_DIN0207_L6.3mm_D2.5mm_P10.16mm_Horizontal, symbol R
- added R4: 33, Resistors_ThroughHole:R_Axial_DIN0207_L6.3mm_D2.5mm_P10.16mm_Horizontal, symbol R
- added R5: 10ohm 225W, Resistors_SMD:R_0201, symbol R
- added SW1, SW2: SWITCH_DPST, Buttons_Switches_SMD:SW_DIP_x2_W5.08mm_Slide_Copal_CHS-A, symbol SWITCH_DPST
- added U1: DS18B20, TO_SOT_Packages_THT:TO-92_Inline_Narrow_Oval, symbol DS18B20
- added U2, U3: D2450, Housings_SIP:SIP4_Sharp-SSR_Pitch7.62mm_Angled, symbol D2450
- added U4: 300XBXC1, Buttons_Switches_SMD:SW_DIP_x4_W8.61mm_Slide_LowProfile, symbol 300XBXC1
- BZ1: renamed from BZ?; footprint (none) -> Buzzers_Beepers:Buzzer_12x9.5RM7.6
- T1: renamed from T?; footprint (none) -> Buttons_Switches_SMD:SW_DIP_x2_W6.15mm_Slide_Omron_A6H
Connections:
- net at T1.1 (AA): now also SW1.2, U2.1
- net at T1.2 (AB): now also SW1.4, SW2.4, U4.8 (B)
- net at T1.3 (SA): now also MCU1.3 (GND), U1.1 (GND)
- net at T1.4 (SB): now also MCU1.4 (+5V), R1.2, U1.3 (VDD)
- net at BZ1.1 (-): now also MCU1.12 (D4)
- net at BZ1.2 (+): now also C1.1, MCU1.10 (GND), R3.1, U2.4, U3.4
- new net: MCU1.13 (D5), U2.3
- new net: MCU1.15 (D7), U3.3
- new net: MCU1.7 (D2/SDA), R1.1, U1.2 (DQ)
- new net: MCU1.9 (+5V), R2.2
- new net: R5.1, SW2.1, U4.3
- new net: P1.2 (Live), SW2.2
- new net: P1.3 (Neutral), SW2.3
- new net: R5.2, U2.2, U3.1, U4.5
- new net: U3.2, U4.7 (A)
- new net CT_CLAMP_INPUT1: MCU1.22 (D18/A0), R4.1
- new net CT_CLAMP_INPUT2: C1.2, R2.1, R3.2, R4.2
- new net MAINS_EARTH: P1.1 (Earth)
- new net MAINS_LIVE: SW1.1
- new net MAINS_NEUTRAL: SW1.3
- no-connect marks 0 -> 14
Other:
- note added: "CT clamp around this wire"
- note added: "Resistor within Industruino"
- note added: "Section within Industruino"
- moved on the sheet: BZ1, T1
